File: OPS.kicad_sch (KiCad schematic)
At the start: 99 parts, among them J1 USB, J2 PWR, J3 Banana, J4 Banana, J5 CON_PWR, J6 CON_DATA, J7 M3, P1 TC2030, Q1 SS8050, Q2 AO3400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

Commit message: update
Connections:
- net GND: now also U4.11 (GND)
Changed lines of the file:
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@@
     (pin "1")
     (pin "10")
+    (pin "11")
     (pin "12")
     (pin "13")
